File: ABL Board/AV Design.brd (EAGLE design)
At the start: 62.2 x 63.5 mm, 32 parts, among them Q1 MMBT4403, U2 LM317, U5 HX711, X1 LOADCELL 3, X2 LOADCELL 2, X3 LOADCELL 1, X4 INPUT, X8 ABL_LED

Commit message: fixed ABL board
Parts:
- moved X4 1.22 mm to (76.5, 45.9), turned to 0 degrees
- moved X8 1.05 mm to (87.5, 45.9), turned to 0 degrees
Routing:
- net SCK: track 0.00 -> 41.7 mm, vias 0 -> 1
- net DOUT: track 31.8 -> 40.0 mm
- net Z_OUT: track 53.3 -> 56.2 mm
- net N$14: track 22.8 -> 21.3 mm
- net GND: track 41.6 -> 43.1 mm
- net 24V: track 69.1 -> 70.4 mm
- net Z_DIR: track 43.8 -> 45.0 mm
- net 12V: track 94.5 -> 94.6 mm, vias 1 -> 2
Other:
- outline, holes or cut-outs redrawn
