File: ABL Board/Julia ABL Board.sch (EAGLE design)
At the start: 32 parts, among them Q1 MMBT4403, U2 LM317, U5 HX711, X1 LOADCELL 3, X2 LOADCELL 2, X3 LOADCELL 1, X4 INPUT, X8 ABL_LED

Commit message: generated ABL board gerbers
Parts:
- added U$2: FRACKTALLOGO, FracktalWorks_Eagle_Library:FRACKTALLOGO
Changed lines of the file:
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@@
 <part name="ZOUT" library="testpad" library_urn="urn:adsk.eagle:library:385" deviceset="TP" device="B2,54" package3d_urn="urn:adsk.eagle:package:27948/1"/>
 <part name="ZDIR" library="testpad" library_urn="urn:adsk.eagle:library:385" deviceset="TP" device="B2,54" package3d_urn="urn:adsk.eagle:package:27948/1"/>
+<part name="U$2" library="FracktalWorks_Eagle_Library" deviceset="FRACKTALLOGO" device=""/>
 </parts>
 <sheets>
@@
 <attribute name="TP_SIGNAL_NAME" x="46.99" y="3.81" size="1.778" layer="97"/>
 </instance>
+<instance part="U$2" gate="G$1" x="-22.86" y="-35.56" smashed="yes"/>
 </instances>
 <busses>

Commit message: Added LED to ABL board
Parts:
- added ABL_LED: (no value), SparkFun-LED:LED-3MM-NO_SILK
Connections:
- net GND: now also ABL_LED.C
- net N$14: now also ABL_LED.A
Changed lines of the file:
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@@
 <setting verticaltext="up"/>
 </settings>
-<grid distance="0.1" unitdist="inch" unit="inch" style="lines" multiple="1" display="no" altdistance="0.01" altunitdist="inch" altunit="inch"/>
+<grid distance="0.01" unitdist="inch" unit="inch" style="lines" multiple="1" display="no" altdistance="0.01" altunitdist="inch" altunit="inch"/>
 <layers>
 <layer number="1" name="Top" color="4" fill="1" visible="no" active="no"/>
@@
 <part name="ZDIR" library="testpad" library_urn="urn:adsk.eagle:library:385" deviceset="TP" device="B2,54" package3d_urn="urn:adsk.eagle:package:27948/1"/>
 <part name="U$2" library="FracktalWorks_Eagle_Library" deviceset="FRACKTALLOGO" device=""/>
+<part name="ABL_LED" library="SparkFun-LED" deviceset="LED" device="-3MM-NO_SILK"/>
+<part name="GND1" library="SparkFun-PowerSymbols" deviceset="GND" device=""/>
 </parts>
 <sheets>
@@
 </instance>
 <instance part="U$2" gate="G$1" x="-22.86" y="-35.56" smashed="yes"/>
+<instance part="ABL_LED" gate="G$1" x="231.14" y="78.74" smashed="yes" rot="R180">
+<attribute name="NAME" x="234.569" y="83.312" size="1.778" layer="95" font="vector" rot="R270"/>
+<attribute name="VALUE" x="229.235" y="83.312" size="1.778" layer="96" font="vector" rot="R270" align="top-left"/>
+</instance>
+<instance part="GND1" gate="1" x="221.4356" y="81.8698" smashed="yes">
+<attribute name="VALUE" x="221.4356" y="81.6158" size="1.778" layer="96" align="top-center"/>
+</instance>
 </instances>
 <busses>
@@
 <wire x1="68.58" y1="63.5" x2="76.2" y2="63.5" width="0.1524" layer="91"/>
 <label x="76.2" y="63.5" size="1.778" layer="95"/>
+</segment>
+<segment>
+<pinref part="ABL_LED" gate="G$1" pin="C"/>
+<wire x1="231.14" y1="83.82" x2="231.14" y2="89.154" width="0.1524" layer="91"/>
+<wire x1="231.14" y1="89.154" x2="221.4356" y2="89.154" width="0.1524" layer="91"/>
+<pinref part="GND1" gate="1" pin="GND"/>
+<wire x1="221.4356" y1="89.154" x2="221.4356" y2="84.4098" width="0.1524" layer="91"/>
 </segment>
 </net>
@@
 <wire x1="246.2276" y1="55.6768" x2="246.2276" y2="77.0892" width="0.1524" layer="91"/>
 <wire x1="246.2276" y1="77.0892" x2="249.8696" y2="77.0892" width="0.1524" layer="91"/>
-</segment>
-</net>
+<pinref part="ABL_LED" gate="G$1" pin="A"/>
+<wire x1="254" y1="43.18" x2="231.14" y2="43.18" width="0.1524" layer="91"/>
+<wire x1="231.14" y1="43.18" x2="231.14" y2="76.2" width="0.1524" layer="91"/>
+</segment>
+</net>
